File: KREWETACM4/Payload_cm4_23/Payload_cm4_23.kicad_sch (KiCad schematic)
At the start: 5 parts

Commit message: updated hardware ELSA and HB
Parts:
- renumbered H1 to H5, H1 to H6, H1 to H7, H1 to H8
