File: KREWETACM4/Payload_cm4_23/power.kicad_sch (KiCad schematic)
At the start: 26 parts, among them IC2 LM66200DRLR, IC3 TPS61023DRLT, IC4 TPS62A02ADRLR, J11 XT30-M

Commit message: updated hardware ELSA and HB
Parts:
- renumbered R5 to R15
