File: KREWETACM4/Payload_cm4_23/rtc.kicad_sch (KiCad schematic)
At the start: 7 parts, among them IC1 RV-3028-C7_32.768kHz_1ppm_TA_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

Commit message: updated hardware ELSA and HB
Parts:
- renumbered R9 to R25, R9 to R26
