File: KREWETACM4/Payload_cm4_23/ssd.kicad_sch (KiCad schematic)
At the start: 5 parts, among them J4 1-2199230-6

Commit message: updated hardware ELSA and HB
Parts:
- renumbered C17 to C10, C17 to C11, C17 to C9, H1 to H9
